File: CANreader-XL.brd (EAGLE design)
At the start: 99.8 x 49.8 mm, 99 parts, among them IC1 STM32F107RBT, IC2 TJA1055T/3, IC3 BD9G101G, IC4 LM1117IMPX-3.3, IC5 MCP2562-SOIC8, IC7 DP83848I, Q1 25MHz, SW1 SLEEP, SW2 TERM, U1 HC_05, X1 ST-USB-009A, X2 SWD, X3 CAN+GPIO, X4 UART

Commit message: Test inital routing
Parts:
- moved LED1 92.7 mm to (96.1, 36.3)
- moved LED2 92.7 mm to (96.1, 46.0)
- moved LED3 92.7 mm to (96.1, 41.1)
- moved R13 81.3 mm to (87.6, 46.0)
- moved R14 81.3 mm to (90.2, 46.0)
- moved R21 81.3 mm to (92.7, 46.0)
- moved R29 34.1 mm to (93.7, 24.1), flipped to the bottom, turned to 0 degrees
- moved R28 31.9 mm to (93.7, 26.7), flipped to the bottom, turned to 0 degrees
- moved C8 23.9 mm to (75.2, 41.1), flipped to the bottom
- moved C28 22.6 mm to (77.2, 41.1), flipped to the bottom, turned to 270 degrees
- moved C30 21.4 mm to (79.2, 41.1), flipped to the bottom, turned to 270 degrees
- moved IC7 10.2 mm to (77.2, 41.1)
- moved SW1 6.99 mm to (77.1, 9.14), turned to 0 degrees
- moved QG1 5.09 mm to (67.3, 45.2), turned to 180 degrees
- moved C5 4.89 mm to (55.1, 36.6), turned to 0 degrees
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Connections:
- removed net N$29: J1.TD-
- net TD-: now also J1.TD-
Routing:
- net RMII_MDC: track 0.00 -> 41.7 mm, vias 0 -> 2
- net RMII_MDIO: track 0.00 -> 39.0 mm, vias 0 -> 2
- net RMII_REF_CLK: track 0.00 -> 37.5 mm, vias 0 -> 2
- net GND: track 888.5 -> 854.0 mm, vias 10 -> 12
- net LED_LINK: track 0.00 -> 32.7 mm, vias 0 -> 1
- net N$15: track 31.7 -> 0.00 mm
- net LEDACT_LINK: track 0.00 -> 30.6 mm, vias 0 -> 1
- net RMII_TXD1: track 0.00 -> 28.6 mm, vias 0 -> 2
- net RMII_TXD0: track 0.00 -> 25.4 mm, vias 0 -> 2
- net TD-: track 0.00 -> 23.1 mm
- net N$10: track 22.8 -> 0.00 mm
- net TD+: track 0.00 -> 22.7 mm
- net RMII_TX_EN: track 0.00 -> 20.2 mm, vias 0 -> 2
- net RMII_CRS_DV: track 0.00 -> 18.7 mm, vias 0 -> 2
- net RD+: track 0.00 -> 18.3 mm
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
Commit message: Fix BT LED
Connections:
- removed net N$15: LED3.A, U1.24
- new net N$5: LED3.A, U1.31
Changed lines of the file:
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@@
 <wire x1="44.26" y1="30.925" x2="47.082" y2="33.548" width="0" layer="19" extent="1-1"/>
-</signal>
-<signal name="N$10">
-<contactref element="U1" pad="32"/>
-<contactref element="LED2" pad="A"/>
-<wire x1="18.24" y1="46.909" x2="96.139" y2="44.704" width="0" layer="19" extent="1-1"/>
 </signal>
 <signal name="N$11">
@@
 <contactref element="R13" pad="2"/>
 <wire x1="87.63" y1="45.024" x2="96.139" y2="47.244" width="0" layer="19" extent="16-16"/>
-</signal>
-<signal name="N$15">
-<contactref element="LED3" pad="A"/>
-<contactref element="U1" pad="24"/>
-<wire x1="30.24" y1="46.909" x2="96.139" y2="39.878" width="0" layer="19" extent="1-1"/>
 </signal>
 <signal name="N$13">
@@
 <wire x1="13.302" y1="12.827" x2="49.582" y2="29.048" width="0" layer="19" extent="1-1"/>
 </signal>
+<signal name="N$5">
+<contactref element="LED3" pad="A"/>
+<contactref element="U1" pad="31"/>
+<wire x1="19.74" y1="46.909" x2="96.139" y2="39.878" width="0" layer="19" extent="1-1"/>
+</signal>
+<signal name="N$10">
+<contactref element="U1" pad="32"/>
+<contactref element="LED2" pad="A"/>
+<wire x1="18.24" y1="46.909" x2="96.139" y2="44.704" width="0" layer="19" extent="1-1"/>
+</signal>
 </signals>
